Commit message: remove pycache and fix package name

File: monospheres/urdf/inspection_geometry.urdf.xacro (robot description, xacro)
@@ -10,5 +10,5 @@
       <origin xyz="0 0 0" rpy="0 0 3.141592653589793"/>
       <geometry>
-        <mesh filename="package://spatial_ai/meshes/inspection_world.dae" scale="2 2 1"/>
+        <mesh filename="package://monospheres/meshes/inspection_world.dae" scale="2 2 1"/>
       </geometry>
     </visual>
@@ -16,5 +16,5 @@
       <origin xyz="0 0 0" rpy="0 0 3.141592653589793"/>
       <geometry>
-        <mesh filename="package://spatial_ai/meshes/inspection_water.dae" scale="2 2 1"/>
+        <mesh filename="package://monospheres/meshes/inspection_water.dae" scale="2 2 1"/>
       </geometry>
     </visual>
@@ -22,5 +22,5 @@
       <origin xyz="0 0 0" rpy="0 0 3.141592653589793"/>
       <geometry>
-        <mesh filename="package://spatial_ai/meshes/inspection_world.dae" scale="2 2 1"/>
+        <mesh filename="package://monospheres/meshes/inspection_world.dae" scale="2 2 1"/>
       </geometry>
       <surface>
